File: hardware/switch-rev2.brd (EAGLE design)
At the start: 94 x 44.5 mm, 100 parts, among them IC1 KS8995MA, IC2 MEGA168-20AU, Y1 12MHz, Y2 25MHz

Commit message: hw: rev2: progress save
todo: fix QFN spacing
Routing:
- net N$69: track 4.79 -> 5.34 mm
Changed lines of the file:
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@@
 <via x="22.5552" y="19.304" extent="1-16" drill="0.508"/>
 <via x="23.9776" y="20.7264" extent="1-16" drill="0.508"/>
-<via x="20.1168" y="31.0896" extent="1-16" drill="0.508"/>
-<via x="20.9296" y="30.2768" extent="1-16" drill="0.508"/>
+<via x="20.32" y="31.0896" extent="1-16" drill="0.508"/>
+<via x="20.32" y="28.0416" extent="1-16" drill="0.508"/>
 <via x="16.0528" y="38.608" extent="1-16" drill="0.508"/>
 <via x="19.5072" y="39.0144" extent="1-16" drill="0.508"/>
-<via x="25.1968" y="26.8224" extent="1-16" drill="0.508"/>
-<via x="25.1968" y="25.4" extent="1-16" drill="0.508"/>
+<via x="24.9936" y="26.6192" extent="1-16" drill="0.508"/>
+<via x="24.9936" y="24.5872" extent="1-16" drill="0.508"/>
 <via x="18.0848" y="31.496" extent="1-16" drill="0.508"/>
 <via x="18.0848" y="30.0736" extent="1-16" drill="0.508"/>
+<via x="37.1856" y="15.24" extent="1-16" drill="0.508"/>
+<via x="38.2016" y="16.256" extent="1-16" drill="0.508"/>
+<via x="39.2176" y="15.24" extent="1-16" drill="0.508"/>
+<via x="38.4048" y="28.6512" extent="1-16" drill="0.508"/>
+<via x="37.3888" y="29.6672" extent="1-16" drill="0.508"/>
+<via x="39.4208" y="29.6672" extent="1-16" drill="0.508"/>
+<via x="19.304" y="21.9456" extent="1-16" drill="0.508"/>
+<via x="20.5232" y="23.5712" extent="1-16" drill="0.508"/>
 </signal>
 <signal name="+5V/1" class="1">
@@
 <contactref element="R61" pad="2"/>
 <contactref element="ETH4" pad="11"/>
-<wire x1="61.214" y1="41.6814" x2="61.214" y2="40.7924" width="0.2032" layer="16"/>
-<wire x1="61.214" y1="40.7924" x2="62.992" y2="39.0144" width="0.2032" layer="16"/>
-<wire x1="62.992" y1="39.0144" x2="62.992" y2="37.6292" width="0.2032" layer="16"/>
+<wire x1="62.992" y1="37.6292" x2="62.992" y2="40.8432" width="0.2032" layer="16"/>
+<wire x1="62.992" y1="40.8432" x2="62.1538" y2="41.6814" width="0.2032" layer="16"/>
+<wire x1="61.214" y1="41.6814" x2="62.1538" y2="41.6814" width="0.2032" layer="16"/>
 </signal>
 <signal name="MODE">
@@
 <contactref element="C24" pad="1"/>
 <contactref element="IC3" pad="3"/>
-<wire x1="6.9704" y1="15.0112" x2="6.9704" y2="15.5848" width="0.4064" layer="1"/>
-<wire x1="6.9704" y1="15.5848" x2="6.7056" y2="15.8496" width="0.4064" layer="1"/>
-<wire x1="6.7056" y1="15.8496" x2="5.8928" y2="15.8496" width="0.4064" layer="1"/>
-<wire x1="5.8928" y1="15.8496" x2="4.4704" y2="17.272" width="0.4064" layer="1"/>
-<wire x1="4.4704" y1="17.272" x2="4.4704" y2="17.8816" width="0.4064" layer="1"/>
-<wire x1="4.4704" y1="17.8816" x2="1.4224" y2="20.9296" width="0.4064" layer="1"/>
-<wire x1="1.4224" y1="20.9296" x2="1.4224" y2="26.284" width="0.4064" layer="1"/>
-<wire x1="1.4224" y1="27.2288" x2="1.4224" y2="33.1216" width="0.4064" layer="1"/>
-<wire x1="1.4224" y1="33.1216" x2="1.966" y2="33.6652" width="0.4064" layer="1"/>
-<wire x1="3.4544" y1="33.6652" x2="1.966" y2="33.6652" width="0.4064" layer="1"/>
-<wire x1="3.4544" y1="26.7564" x2="1.8948" y2="26.7564" width="0.4064" layer="1"/>
-<wire x1="1.8948" y1="26.7564" x2="1.4224" y2="27.2288" width="0.4064" layer="1"/>
-<wire x1="1.4224" y1="26.284" x2="1.8948" y2="26.7564" width="0.4064" layer="1"/>
-<wire x1="3.4544" y1="26.7564" x2="4.8108" y2="26.7564" width="0.4064" layer="1"/>
-<wire x1="4.8108" y1="26.7564" x2="4.8768" y2="26.8224" width="0.4064" layer="1"/>
-<wire x1="3.4544" y1="33.6652" x2="4.8108" y2="33.6652" width="0.4064" layer="1"/>
-<wire x1="4.8108" y1="33.6652" x2="4.8768" y2="33.7312" width="0.4064" layer="1"/>
+<wire x1="6.9704" y1="15.0112" x2="6.9704" y2="15.5848" width="0.6096" layer="1"/>
+<wire x1="6.9704" y1="15.5848" x2="6.7056" y2="15.8496" width="0.6096" layer="1"/>
+<wire x1="6.7056" y1="15.8496" x2="5.8928" y2="15.8496" width="0.6096" layer="1"/>
+<wire x1="5.8928" y1="15.8496" x2="4.4704" y2="17.272" width="0.6096" layer="1"/>
+<wire x1="4.4704" y1="17.272" x2="4.4704" y2="17.8816" width="0.6096" layer="1"/>
+<wire x1="4.4704" y1="17.8816" x2="1.4224" y2="20.9296" width="0.6096" layer="1"/>
+<wire x1="1.4224" y1="20.9296" x2="1.4224" y2="26.284" width="0.6096" layer="1"/>
+<wire x1="1.4224" y1="27.2288" x2="1.4224" y2="33.1216" width="0.6096" layer="1"/>
+<wire x1="1.4224" y1="33.1216" x2="1.966" y2="33.6652" width="0.6096" layer="1"/>
+<wire x1="3.4544" y1="33.6652" x2="1.966" y2="33.6652" width="0.6096" layer="1"/>
+<wire x1="3.4544" y1="26.7564" x2="1.8948" y2="26.7564" width="0.6096" layer="1"/>
+<wire x1="1.8948" y1="26.7564" x2="1.4224" y2="27.2288" width="0.6096" layer="1"/>
+<wire x1="1.4224" y1="26.284" x2="1.8948" y2="26.7564" width="0.6096" layer="1"/>
+<wire x1="3.4544" y1="26.7564" x2="4.8108" y2="26.7564" width="0.6096" layer="1"/>
+<wire x1="4.8108" y1="26.7564" x2="4.8768" y2="26.8224" width="0.6096" layer="1"/>
+<wire x1="3.4544" y1="33.6652" x2="4.8108" y2="33.6652" width="0.6096" layer="1"/>
+<wire x1="4.8108" y1="33.6652" x2="4.8768" y2="33.7312" width="0.6096" layer="1"/>
 <via x="4.8768" y="33.7312" extent="1-16" drill="0.508"/>
 <via x="4.8768" y="26.8224" extent="1-16" drill="0.508"/>
-<wire x1="3.2004" y1="26.8986" x2="4.8006" y2="26.8986" width="0.4064" layer="16"/>
-<wire x1="4.8006" y1="26.8986" x2="4.8768" y2="26.8224" width="0.4064" layer="16"/>
-<wire x1="3.2004" y1="33.8074" x2="4.8006" y2="33.8074" width="0.4064" layer="16"/>
-<wire x1="4.8006" y1="33.8074" x2="4.8768" y2="33.7312" width="0.4064" layer="16"/>
+<wire x1="3.2004" y1="26.8986" x2="4.8006" y2="26.8986" width="0.6096" layer="16"/>
+<wire x1="4.8006" y1="26.8986" x2="4.8768" y2="26.8224" width="0.6096" layer="16"/>
+<wire x1="3.2004" y1="33.8074" x2="4.8006" y2="33.8074" width="0.6096" layer="16"/>
+<wire x1="4.8006" y1="33.8074" x2="4.8768" y2="33.7312" width="0.6096" layer="16"/>
 </signal>
 <signal name="N$17">

Commit message: hw: rev2: change atmega QFN package
Parts:
- removed IC2: MEGA168-20AU, atmel:MLF32
- added IC5: ATMEGA168-MU, balto:MLF32-TH
Connections:
- net +5V: now also IC5.18, IC5.4, IC5.6; no longer IC2.18, IC2.4, IC2.6
- net CS: now also IC5.14; no longer IC2.14
- net DM: now also IC5.31; no longer IC2.31
- net DP: now also IC5.32; no longer IC2.32
- net GND: now also IC5.21, IC5.3, IC5.5, IC5.TH; no longer IC2.21, IC2.3, IC2.5
- net MISO: now also IC5.16; no longer IC2.16
- net MODE: now also IC5.1; no longer IC2.1
- net MOSI: now also IC5.15; no longer IC2.15
- net SCK: now also IC5.17; no longer IC2.17
- net STATUS: now also IC5.2; no longer IC2.2
- net SW-RESET: now also IC5.24; no longer IC2.24
- net UC-RESET: now also IC5.29; no longer IC2.29
- net XTAL1: now also IC5.7; no longer IC2.7
- net XTAL2: now also IC5.8; no longer IC2.8
Routing:
- net GND: track 0.00 -> 5.73 mm
Changed lines of the file:
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@@
 <elements>
 <element name="IC1" library="micrel" package="PQFP128L" value="KS8995MA" x="24.9936" y="22.5552" rot="R90"/>
-<element name="IC2" library="atmel" package="MLF32" value="MEGA168-20AU" x="18.0848" y="4.6736" rot="R45"/>
 <element name="C1" library="rcl" package="C0805" value=".1u" x="20.1168" y="25.8064" rot="MR180"/>
 <element name="R1" library="rcl" package="R0603" value="3.01K 1%" x="26.6192" y="22.352" rot="MR180"/>
@@
 <element name="BOX1" library="hammond" package="1591XXA" value="HAMMOND-BOX-XXA" x="0" y="0" locked="yes"/>
 <element name="D2" library="diode" package="SMB" value="" x="26.0096" y="41.2496" rot="MR0"/>
+<element name="IC5" library="balto" package="MLF32-TH" value="ATMEGA168-MU" x="18.0848" y="4.6736" rot="R45"/>
 </elements>
 <signals>
@@
 <contactref element="C3" pad="2"/>
 <contactref element="R23" pad="1"/>
-<contactref element="IC2" pad="3"/>
-<contactref element="IC2" pad="5"/>
-<contactref element="IC2" pad="21"/>
 <contactref element="C1" pad="2"/>
 <contactref element="C5" pad="2"/>
@@
 <via x="19.304" y="21.9456" extent="1-16" drill="0.508"/>
 <via x="20.5232" y="23.5712" extent="1-16" drill="0.508"/>
+<contactref element="IC5" pad="3"/>
+<contactref element="IC5" pad="TH"/>
+<contactref element="IC5" pad="5"/>
+<contactref element="IC5" pad="3"/>
+<contactref element="IC5" pad="TH"/>
+<contactref element="IC5" pad="5"/>
+<contactref element="IC5" pad="21"/>
+<wire x1="15.89276875" y1="3.542228125" x2="16.8656" y2="4.515059375" width="0.254" layer="1"/>
+<wire x1="16.8656" y1="4.515059375" x2="16.8656" y2="4.6736" width="0.254" layer="1"/>
+<wire x1="16.599875" y1="2.835121875" x2="18.0848" y2="4.320046875" width="0.254" layer="1"/>
+<wire x1="18.0848" y1="4.320046875" x2="18.0848" y2="4.6736" width="0.254" layer="1"/>
+<wire x1="19.569721875" y1="6.512075" x2="18.950446875" y2="5.8928" width="0.254" layer="1"/>
+<wire x1="18.950446875" y1="5.8928" x2="18.0848" y2="5.8928" width="0.254" layer="1"/>
 </signal>
 <signal name="+5V/1" class="1">
@@
 <contactref element="IC1" pad="77"/>
 <contactref element="IC1" pad="100"/>
-<contactref element="IC2" pad="6"/>
-<contactref element="IC2" pad="4"/>
-<contactref element="IC2" pad="18"/>
 <contactref element="C1" pad="1"/>
 <contactref element="C5" pad="1"/>
@@
 <wire x1="21.1328" y1="32.512" x2="19.8476" y2="33.7972" width="0.4064" layer="16"/>
 <wire x1="18.8976" y1="33.7972" x2="19.8476" y2="33.7972" width="0.4064" layer="16"/>
+<contactref element="IC5" pad="4"/>
+<contactref element="IC5" pad="6"/>
+<contactref element="IC5" pad="18"/>
 </signal>
 <signal name="+5V/2" class="1">
@@
 <signal name="CS">
 <contactref element="IC1" pad="112"/>
-<contactref element="IC2" pad="14"/>
 <wire x1="20.276828125" y1="3.542228125" x2="20.77105625" y2="3.048" width="0.2032" layer="1"/>
 <wire x1="20.77105625" y1="3.048" x2="22.1488" y2="3.048" width="0.2032" layer="1"/>
 <wire x1="23.2436" y1="10.9552" x2="23.2436" y2="4.1428" width="0.2032" layer="1"/>
 <wire x1="23.2436" y1="4.1428" x2="22.1488" y2="3.048" width="0.2032" layer="1"/>
+<contactref element="IC5" pad="14"/>
 </signal>
 <signal name="SCK">
 <contactref element="IC1" pad="110"/>
-<contactref element="IC2" pad="17"/>
 <contactref element="ISP" pad="3"/>
 <wire x1="22.2436" y1="10.9552" x2="22.2436" y2="8.426" width="0.2032" layer="1"/>
@@
 <wire x1="27.0256" y1="2.6416" x2="25.8064" y2="3.8608" width="0.2032" layer="16"/>
 <wire x1="25.8064" y1="3.8608" x2="24.1808" y2="3.8608" width="0.2032" layer="16"/>
+<contactref element="IC5" pad="17"/>
 </signal>
 <signal name="MOSI">
 <contactref element="IC1" pad="111"/>
-<contactref element="IC2" pad="15"/>
 <contactref element="ISP" pad="4"/>
 <wire x1="22.7436" y1="10.9552" x2="22.7436" y2="7.3004" width="0.2032" layer="1"/>
@@
 <wire x1="21.9456" y1="3.4544" x2="22.7436" y2="4.2524" width="0.2032" layer="1"/>
 <wire x1="22.7436" y1="4.2524" x2="22.7436" y2="6.5172" width="0.2032" layer="1"/>
+<contactref element="IC5" pad="15"/>
 </signal>
 <signal name="MISO">
 <contactref element="IC1" pad="109"/>
-<contactref element="IC2" pad="16"/>
 <contactref element="ISP" pad="1"/>
 <wire x1="20.9839375" y1="4.249334375" x2="21.408203125" y2="4.6736" width="0.2032" layer="1"/>
@@
 <wire x1="21.1328" y1="8.9408" x2="21.1328" y2="5.4864" width="0.2032" layer="16"/>
 <wire x1="21.1328" y1="5.4864" x2="21.9456" y2="4.6736" width="0.2032" layer="16"/>
+<contactref element="IC5" pad="16"/>
 </signal>
 <signal name="N$1">
@@
 <wire x1="23.5712" y1="12.8016" x2="24.5872" y2="12.8016" width="0.2032" layer="16"/>
 <wire x1="24.7436" y1="12.6452" x2="24.7436" y2="10.9552" width="0.2032" layer="1"/>
-<contactref element="IC2" pad="24"/>
 <wire x1="19.1008" y1="8.9408" x2="19.1008" y2="8.164475" width="0.2032" layer="1"/>
 <wire x1="19.1008" y1="8.164475" x2="18.5090625" y2="7.5727375" width="0.2032" layer="1"/>
+<contactref element="IC5" pad="24"/>
 </signal>
 <signal name="UC-RESET">
-<contactref element="IC2" pad="29"/>
 <contactref element="ISP" pad="5"/>
 <wire x1="17.4752" y1="8.5344" x2="18.0848" y2="8.5344" width="0.2032" layer="1"/>
 <via x="18.0848" y="8.5344" extent="1-16" drill="0.508"/>
-<wire x1="16.246321875" y1="6.158521875" x2="15.8496" y2="6.55524375" width="0.2032" layer="1"/>
 <wire x1="15.8496" y1="6.55524375" x2="15.8496" y2="6.9088" width="0.2032" layer="1"/>
 <wire x1="15.8496" y1="6.9088" x2="17.4752" y2="8.5344" width="0.2032" layer="1"/>
@@
 <wire x1="20.7264" y1="8.128" x2="20.32" y2="8.5344" width="0.2032" layer="16"/>
 <wire x1="20.32" y1="8.5344" x2="18.0848" y2="8.5344" width="0.2032" layer="16"/>
+<contactref element="IC5" pad="29"/>
+<wire x1="16.246321875" y1="6.158521875" x2="15.8496" y2="6.55524375" width="0.2032" layer="1"/>
 </signal>
 <signal name="STATUS">
 <contactref element="LED1" pad="A"/>
-<contactref element="IC2" pad="2"/>
 <wire x1="14.144728125" y1="2.51766875" x2="14.1611" y2="2.51766875" width="0.2032" layer="1"/>
 <wire x1="14.1611" y1="2.51766875" x2="15.5392125" y2="3.89578125" width="0.2032" layer="1"/>
+<contactref element="IC5" pad="2"/>
 </signal>
 <signal name="N$47">
@@
 <contactref element="S1" pad="1"/>
 <contactref element="S1" pad="2"/>
-<contactref element="IC2" pad="1"/>
 <wire x1="5.4864" y1="8.5344" x2="2.8448" y2="8.5344" width="0.2032" layer="16"/>
 <wire x1="2.8448" y1="8.5344" x2="1.2192" y2="10.16" width="0.2032" layer="16"/>
@@
 <wire x1="14.1224" y1="38.735" x2="10.6934" y2="38.735" width="0.2032" layer="1"/>
 <wire x1="10.6934" y1="38.735" x2="10.5664" y2="38.608" width="0.2032" layer="1"/>
+<contactref element="IC5" pad="1"/>
 </signal>
 <signal name="V_USB">
@@
 <signal name="DP">
 <contactref element="R16" pad="1"/>
-<contactref element="IC2" pad="32"/>
 <wire x1="15.185659375" y1="5.0978625" x2="14.797121875" y2="5.4864" width="0.2032" layer="1"/>
-<wire x1="14.797121875" y1="5.4864" x2="14.4272" y2="5.4864" width="0.2032" layer="1"/>
-<wire x1="14.4272" y1="5.4864" x2="14.224" y2="5.2832" width="0.2032" layer="1"/>
-<via x="14.224" y="5.2832" extent="1-16" drill="0.508"/>
-<wire x1="14.224" y1="5.2832" x2="13.0048" y2="5.2832" width="0.2032" layer="16"/>
+<wire x1="14.797121875" y1="5.4864" x2="14.3256" y2="5.4864" width="0.2032" layer="1"/>
+<wire x1="14.3256" y1="5.4864" x2="14.1224" y2="5.2832" width="0.2032" layer="1"/>
+<via x="14.1224" y="5.2832" extent="1-16" drill="0.508"/>
+<wire x1="14.1224" y1="5.2832" x2="13.0048" y2="5.2832" width="0.2032" layer="16"/>
 <wire x1="13.0048" y1="5.2832" x2="10.3632" y2="7.9248" width="0.2032" layer="16"/>
 <wire x1="10.3632" y1="7.9248" x2="10.3632" y2="10.16" width="0.2032" layer="16"/>
@@
 <via x="9.9568" y="10.5664" extent="1-16" drill="0.508"/>
 <wire x1="10.3632" y1="10.16" x2="9.9568" y2="10.5664" width="0.2032" layer="16"/>
+<contactref element="IC5" pad="32"/>
 </signal>
 <signal name="DM">
 <contactref element="R15" pad="1"/>
-<contactref element="IC2" pad="31"/>
 <wire x1="15.5392125" y1="5.451415625" x2="14.691428125" y2="6.2992" width="0.2032" layer="1"/>
 <wire x1="14.691428125" y1="6.2992" x2="13.208" y2="6.2992" width="0.2032" layer="1"/>
@@
 <via x="10.9728" y="11.3792" extent="1-16" drill="0.508"/>
 <wire x1="10.9728" y1="8.3312" x2="10.9728" y2="11.3792" width="0.2032" layer="16"/>
+<contactref element="IC5" pad="31"/>
 </signal>
 <signal name="N$16">
@@
 </signal>
 <signal name="XTAL1">
-<contactref element="IC2" pad="7"/>
 <contactref element="Y1" pad="1"/>
 <contactref element="C23" pad="1"/>
@@
 <wire x1="11.9888" y1="2.6416" x2="11.9888" y2="3.6576" width="0.2032" layer="1"/>
 <wire x1="11.9888" y1="3.6576" x2="11.176" y2="4.4704" width="0.2032" layer="1"/>
+<contactref element="IC5" pad="7"/>
 </signal>
 <signal name="XTAL2">
-<contactref element="IC2" pad="8"/>
 <contactref element="Y1" pad="3"/>
 <contactref element="C21" pad="1"/>
@@
 <wire x1="11.1068" y1="2.214" x2="11.8068" y2="2.214" width="0.2032" layer="1"/>
 <wire x1="11.8068" y1="2.214" x2="12.8016" y2="1.2192" width="0.2032" layer="1"/>
+<contactref element="IC5" pad="8"/>
 </signal>
 </signals>
